Commit message: Started End-effector URDF

File: ros2_system/src/motion_control_module/urdf/end_effector.urdf.xacro (robot description, xacro)
@@ -3,35 +3,34 @@
   <!--
     End-effector attachment for UR5e
-    This adds a visual representation of a gripper/tool to the robot
+    Tongs/Scissors-style gripper with two prongs
   -->
   <xacro:macro name="end_effector" params="prefix">
-    <!-- End-effector link -->
+    <!-- Base/Pivot link (connection point) -->
     <link name="${prefix}end_effector_link">
       <visual>
-        <origin xyz="0 0 0.075" rpy="0 0 0"/>
-        <geometry>
-          <!-- Placeholder: Simple box representing gripper/tool -->
-          <!-- Dimensions: 8cm wide x 6cm deep x 15cm long -->
-          <box size="0.08 0.06 0.15"/>
-        </geometry>
-        <material name="end_effector_material">
-          <color rgba="0.8 0.3 0.1 1.0"/>  <!-- Orange color -->
-        </material>
-      </visual>
-      <collision>
-        <origin xyz="0 0 0.075" rpy="0 0 0"/>
-        <geometry>
-          <box size="0.08 0.06 0.15"/>
-        </geometry>
-      </collision>
-      <inertial>
-        <origin xyz="0 0 0.075" rpy="0 0 0"/>
-        <mass value="0.5"/>  <!-- Placeholder mass: 500g -->
-        <inertia ixx="0.001" ixy="0.0" ixz="0.0"
-                 iyy="0.001" iyz="0.0"
-                 izz="0.001"/>
-      </inertial>
-    </link>
-    <!-- Joint connecting tool0 to end-effector -->
+        <origin xyz="0 0 0.02" rpy="0 0 0"/>
+        <geometry>
+          <!-- Base mount - small cylinder -->
+          <cylinder radius="0.025" length="0.04"/>
+        </geometry>
+        <material name="base_material">
+          <color rgba="0.2 0.2 0.2 1.0"/>  <!-- Dark gray -->
+        </material>
+      </visual>
+      <collision>
+        <origin xyz="0 0 0.02" rpy="0 0 0"/>
+        <geometry>
+          <cylinder radius="0.025" length="0.04"/>
+        </geometry>
+      </collision>
+      <inertial>
+        <origin xyz="0 0 0.05" rpy="0 0 0"/>
+        <mass value="0.3"/>
+        <inertia ixx="0.0005" ixy="0.0" ixz="0.0"
+                 iyy="0.0005" iyz="0.0"
+                 izz="0.0005"/>
+      </inertial>
+    </link>
+    <!-- Joint connecting tool0 to end-effector base -->
     <joint name="${prefix}end_effector_joint" type="fixed">
       <parent link="${prefix}tool0"/>
@@ -39,38 +38,171 @@
       <origin xyz="0 0 0" rpy="0 0 0"/>
     </joint>
-    <!-- Optional: Add gripper fingers visualization -->
-    <link name="${prefix}gripper_left_finger">
-      <visual>
-        <origin xyz="0 0.02 0.14" rpy="0 0 0"/>
-        <geometry>
-          <box size="0.02 0.01 0.08"/>
-        </geometry>
-        <material name="finger_material">
-          <color rgba="0.3 0.3 0.3 1.0"/>  <!-- Dark gray -->
-        </material>
-      </visual>
-    </link>
-    <joint name="${prefix}gripper_left_finger_joint" type="fixed">
+    <!-- Left arm - Upper limb (first segment) -->
+    <link name="${prefix}gripper_left_upper">
+      <visual>
+        <origin xyz="0 0.015 0.03" rpy="0 0 0"/>
+        <geometry>
+          <box size="0.015 0.022 0.06"/>  <!-- Upper segment -->
+        </geometry>
+        <material name="prong_material">
+          <color rgba="0.7 0.7 0.7 1.0"/>  <!-- Light gray -->
+        </material>
+      </visual>
+      <collision>
+        <origin xyz="0 0.015 0.03" rpy="0 0 0"/>
+        <geometry>
+          <box size="0.015 0.022 0.06"/>
+        </geometry>
+      </collision>
+      <inertial>
+        <origin xyz="0 0.015 0.03" rpy="0 0 0"/>
+        <mass value="0.05"/>
+        <inertia ixx="0.00005" ixy="0.0" ixz="0.0"
+                 iyy="0.00005" iyz="0.0"
+                 izz="0.000005"/>
+      </inertial>
+    </link>
+    <joint name="${prefix}gripper_left_upper_joint" type="fixed">
       <parent link="${prefix}end_effector_link"/>
-      <child link="${prefix}gripper_left_finger"/>
-      <origin xyz="0 0 0" rpy="0 0 0"/>
-    </joint>
-    <link name="${prefix}gripper_right_finger">
-      <visual>
-        <origin xyz="0 -0.02 0.14" rpy="0 0 0"/>
-        <geometry>
-          <box size="0.02 0.01 0.08"/>
-        </geometry>
-        <material name="finger_material">
-          <color rgba="0.3 0.3 0.3 1.0"/>  <!-- Dark gray -->
-        </material>
-      </visual>
-    </link>
-    <joint name="${prefix}gripper_right_finger_joint" type="fixed">
+      <child link="${prefix}gripper_left_upper"/>
+      <origin xyz="0 0 0.04" rpy="0 0 0"/>
+    </joint>
+    <!-- Left arm - Lower limb (second segment) -->
+    <link name="${prefix}gripper_left_lower">
+      <visual>
+        <origin xyz="0 0.015 0.03" rpy="0 0 0"/>
+        <geometry>
+          <box size="0.012 0.018 0.06"/>  <!-- Lower segment, slightly thinner -->
+        </geometry>
+        <material name="prong_material">
+          <color rgba="0.7 0.7 0.7 1.0"/>  <!-- Light gray -->
+        </material>
+      </visual>
+      <collision>
+        <origin xyz="0 0.015 0.03" rpy="0 0 0"/>
+        <geometry>
+          <box size="0.012 0.018 0.06"/>
+        </geometry>
+      </collision>
+      <inertial>
+        <origin xyz="0 0.015 0.03" rpy="0 0 0"/>
+        <mass value="0.04"/>
+        <inertia ixx="0.00004" ixy="0.0" ixz="0.0"
+                 iyy="0.00004" iyz="0.0"
+                 izz="0.000004"/>
+      </inertial>
+    </link>
+    <joint name="${prefix}gripper_left_lower_joint" type="fixed">
+      <parent link="${prefix}gripper_left_upper"/>
+      <child link="${prefix}gripper_left_lower"/>
+      <origin xyz="0 0 0.06" rpy="0 0 0"/>  <!-- Offset from upper limb -->
+    </joint>
+    <!-- Left arm tip (tapered end) -->
+    <link name="${prefix}gripper_left_tip">
+      <visual>
+        <origin xyz="0 0.015 0.07" rpy="0 0 0"/>
+        <geometry>
+          <box size="0.01 0.015 0.02"/>  <!-- Smaller tip -->
+        </geometry>
+        <material name="tip_material">
+          <color rgba="0.5 0.5 0.5 1.0"/>  <!-- Medium gray -->
+        </material>
+      </visual>
+      <collision>
+        <origin xyz="0 0.015 0.07" rpy="0 0 0"/>
+        <geometry>
+          <box size="0.01 0.015 0.02"/>
+        </geometry>
+      </collision>
+    </link>
+    <joint name="${prefix}gripper_left_tip_joint" type="fixed">
+      <parent link="${prefix}gripper_left_lower"/>
+      <child link="${prefix}gripper_left_tip"/>
+      <origin xyz="0 0 0.06" rpy="0 0 0"/>  <!-- At end of lower limb -->
+    </joint>
+    <!-- Right arm - Upper limb (first segment) -->
+    <link name="${prefix}gripper_right_upper">
+      <visual>
+        <origin xyz="0 -0.015 0.03" rpy="0 0 0"/>
+        <geometry>
+          <box size="0.015 0.022 0.06"/>  <!-- Upper segment -->
+        </geometry>
+        <material name="prong_material">
+          <color rgba="0.7 0.7 0.7 1.0"/>  <!-- Light gray -->
+        </material>
+      </visual>
+      <collision>
+        <origin xyz="0 -0.015 0.03" rpy="0 0 0"/>
+        <geometry>
+          <box size="0.015 0.022 0.06"/>
+        </geometry>
+      </collision>
+      <inertial>
+        <origin xyz="0 -0.015 0.03" rpy="0 0 0"/>
+        <mass value="0.05"/>
+        <inertia ixx="0.00005" ixy="0.0" ixz="0.0"
+                 iyy="0.00005" iyz="0.0"
+                 izz="0.000005"/>
+      </inertial>
+    </link>
+    <joint name="${prefix}gripper_right_upper_joint" type="fixed">
       <parent link="${prefix}end_effector_link"/>
-      <child link="${prefix}gripper_right_finger"/>
-      <origin xyz="0 0 0" rpy="0 0 0"/>
-    </joint>
-    <!-- Tip frame for easy reference -->
+      <child link="${prefix}gripper_right_upper"/>
+      <origin xyz="0 0 0.04" rpy="0 0 0"/>
+    </joint>
+    <!-- Right arm - Lower limb (second segment) -->
+    <link name="${prefix}gripper_right_lower">
+      <visual>
+        <origin xyz="0 -0.015 0.03" rpy="0 0 0"/>
+        <geometry>
+          <box size="0.012 0.018 0.06"/>  <!-- Lower segment, slightly thinner -->
+        </geometry>
+        <material name="prong_material">
+          <color rgba="0.7 0.7 0.7 1.0"/>  <!-- Light gray -->
+        </material>
+      </visual>
+      <collision>
+        <origin xyz="0 -0.015 0.03" rpy="0 0 0"/>
+        <geometry>
+          <box size="0.012 0.018 0.06"/>
+        </geometry>
+      </collision>
+      <inertial>
+        <origin xyz="0 -0.015 0.03" rpy="0 0 0"/>
+        <mass value="0.04"/>
+        <inertia ixx="0.00004" ixy="0.0" ixz="0.0"
+                 iyy="0.00004" iyz="0.0"
+                 izz="0.000004"/>
+      </inertial>
+    </link>
+    <joint name="${prefix}gripper_right_lower_joint" type="fixed">
+      <parent link="${prefix}gripper_right_upper"/>
+      <child link="${prefix}gripper_right_lower"/>
+      <origin xyz="0 0 0.06" rpy="0 0 0"/>  <!-- Offset from upper limb -->
+    </joint>
+    <!-- Right arm tip (tapered end) -->
+    <link name="${prefix}gripper_right_tip">
+      <visual>
+        <origin xyz="0 -0.015 0.07" rpy="0 0 0"/>
+        <geometry>
+          <box size="0.01 0.015 0.02"/>  <!-- Smaller tip -->
+        </geometry>
+        <material name="tip_material">
+          <color rgba="0.5 0.5 0.5 1.0"/>  <!-- Medium gray -->
+        </material>
+      </visual>
+      <collision>
+        <origin xyz="0 -0.015 0.07" rpy="0 0 0"/>
+        <geometry>
+          <box size="0.01 0.015 0.02"/>
+        </geometry>
+      </collision>
+    </link>
+    <joint name="${prefix}gripper_right_tip_joint" type="fixed">
+      <parent link="${prefix}gripper_right_lower"/>
+      <child link="${prefix}gripper_right_tip"/>
+      <origin xyz="0 0 0.06" rpy="0 0 0"/>  <!-- At end of lower limb -->
+    </joint>
+    <!-- Tip frame for easy reference (center between prongs) -->
     <link name="${prefix}end_effector_tip"/>
     <joint name="${prefix}end_effector_tip_joint" type="fixed">

File: ros2_system/src/motion_control_module/urdf/ur5e_with_end_effector.urdf.xacro (robot description, xacro)
@@ -1,13 +1,48 @@
 <?xml version="1.0"?>
 <robot xmlns:xacro="http://www.ros.org/wiki/xacro" name="ur5e_with_end_effector">
-  <!-- Parameters -->
-  <xacro:arg name="robot_ip" default="192.168.1.102"/>
+  <!-- robot name parameter -->
+  <xacro:arg name="name" default="ur"/>
+  <!-- possible 'ur_type' values: ur3, ur3e, ur5, ur5e, ur10, ur10e, ur16e -->
+  <xacro:arg name="ur_type" default="ur5e"/>
+  <!-- parameters -->
+  <xacro:arg name="tf_prefix" default="" />
   <xacro:arg name="joint_limit_params" default="$(find ur_description)/config/ur5e/joint_limits.yaml"/>
   <xacro:arg name="kinematics_params" default="$(find ur_description)/config/ur5e/default_kinematics.yaml"/>
   <xacro:arg name="physical_params" default="$(find ur_description)/config/ur5e/physical_parameters.yaml"/>
   <xacro:arg name="visual_params" default="$(find ur_description)/config/ur5e/visual_parameters.yaml"/>
-  <xacro:arg name="name" default="ur"/>
-  <xacro:arg name="ur_type" default="ur5e"/>
-  <xacro:arg name="prefix" default=""/>
+  <xacro:arg name="transmission_hw_interface" default=""/>
+  <xacro:arg name="safety_limits" default="false"/>
+  <xacro:arg name="safety_pos_margin" default="0.15"/>
+  <xacro:arg name="safety_k_position" default="20"/>
+  <!-- ros2_control related parameters -->
+  <xacro:arg name="headless_mode" default="false" />
+  <xacro:arg name="robot_ip" default="0.0.0.0" />
+  <xacro:arg name="script_filename" default=""/>
+  <xacro:arg name="output_recipe_filename" default=""/>
+  <xacro:arg name="input_recipe_filename" default=""/>
+  <xacro:arg name="reverse_ip" default="0.0.0.0"/>
+  <xacro:arg name="script_command_port" default="50004"/>
+  <!-- tool communication related parameters-->
+  <xacro:arg name="use_tool_communication" default="false" />
+  <xacro:arg name="tool_voltage" default="0" />
+  <xacro:arg name="tool_parity" default="0" />
+  <xacro:arg name="tool_baud_rate" default="115200" />
+  <xacro:arg name="tool_stop_bits" default="1" />
+  <xacro:arg name="tool_rx_idle_chars" default="1.5" />
+  <xacro:arg name="tool_tx_idle_chars" default="3.5" />
+  <xacro:arg name="tool_device_name" default="/tmp/ttyUR" />
+  <xacro:arg name="tool_tcp_port" default="54321" />
+  <!-- Simulation parameters -->
+  <xacro:arg name="use_fake_hardware" default="false" />
+  <xacro:arg name="fake_sensor_commands" default="false" />
+  <xacro:arg name="sim_gazebo" default="false" />
+  <xacro:arg name="sim_ignition" default="false" />
+  <xacro:arg name="simulation_controllers" default="" />
+  <!-- Network configuration -->
+  <xacro:arg name="reverse_port" default="50001"/>
+  <xacro:arg name="script_sender_port" default="50002"/>
+  <xacro:arg name="trajectory_port" default="50003"/>
+  <xacro:arg name="non_blocking_read" default="false"/>
+  <xacro:arg name="keep_alive_count" default="2"/>
   <!-- Include the base UR macro -->
   <xacro:include filename="$(find ur_description)/urdf/ur_macro.xacro"/>
@@ -19,5 +54,5 @@
   <xacro:ur_robot
     name="$(arg name)"
-    tf_prefix="$(arg prefix)"
+    tf_prefix="$(arg tf_prefix)"
     parent="world"
     joint_limits_parameters_file="$(arg joint_limit_params)"
@@ -25,11 +60,37 @@
     physical_parameters_file="$(arg physical_params)"
     visual_parameters_file="$(arg visual_params)"
-    transmission_hw_interface="hardware_interface/PositionJointInterface"
-    safety_limits="false"
-    safety_pos_margin="0.15"
-    safety_k_position="20">
+    transmission_hw_interface="$(arg transmission_hw_interface)"
+    safety_limits="$(arg safety_limits)"
+    safety_pos_margin="$(arg safety_pos_margin)"
+    safety_k_position="$(arg safety_k_position)"
+    use_fake_hardware="$(arg use_fake_hardware)"
+    fake_sensor_commands="$(arg fake_sensor_commands)"
+    sim_gazebo="$(arg sim_gazebo)"
+    sim_ignition="$(arg sim_ignition)"
+    headless_mode="$(arg headless_mode)"
+    use_tool_communication="$(arg use_tool_communication)"
+    tool_voltage="$(arg tool_voltage)"
+    tool_parity="$(arg tool_parity)"
+    tool_baud_rate="$(arg tool_baud_rate)"
+    tool_stop_bits="$(arg tool_stop_bits)"
+    tool_rx_idle_chars="$(arg tool_rx_idle_chars)"
+    tool_tx_idle_chars="$(arg tool_tx_idle_chars)"
+    tool_device_name="$(arg tool_device_name)"
+    tool_tcp_port="$(arg tool_tcp_port)"
+    robot_ip="$(arg robot_ip)"
+    script_filename="$(arg script_filename)"
+    output_recipe_filename="$(arg output_recipe_filename)"
+    input_recipe_filename="$(arg input_recipe_filename)"
+    reverse_ip="$(arg reverse_ip)"
+    script_command_port="$(arg script_command_port)"
+    reverse_port="$(arg reverse_port)"
+    script_sender_port="$(arg script_sender_port)"
+    trajectory_port="$(arg trajectory_port)"
+    non_blocking_read="$(arg non_blocking_read)"
+    keep_alive_count="$(arg keep_alive_count)"
+    >
     <origin xyz="0 0 0" rpy="0 0 0" />
   </xacro:ur_robot>
   <!-- Attach the end-effector -->
-  <xacro:end_effector prefix="$(arg prefix)"/>
+  <xacro:end_effector prefix="$(arg tf_prefix)"/>
 </robot>

Commit message: end_effector.urdf.xacro

File: ros2_system/src/motion_control_module/urdf/end_effector.urdf.xacro (robot description, xacro)
@@ -41,5 +41,5 @@
     <link name="${prefix}gripper_left_upper">
       <visual>
-        <origin xyz="0 0.015 0.03" rpy="0 0 0"/>
+        <origin xyz="0 0 0.03" rpy="0 0 0"/>  <!-- Center of 6cm box -->
         <geometry>
           <box size="0.015 0.022 0.06"/>  <!-- Upper segment -->
@@ -50,5 +50,5 @@
       </visual>
       <collision>
-        <origin xyz="0 0.015 0.03" rpy="0 0 0"/>
+        <origin xyz="0 0 0.03" rpy="0 0 0"/>
         <geometry>
           <box size="0.015 0.022 0.06"/>
@@ -56,5 +56,5 @@
       </collision>
       <inertial>
-        <origin xyz="0 0.015 0.03" rpy="0 0 0"/>
+        <origin xyz="0 0 0.03" rpy="0 0 0"/>
         <mass value="0.05"/>
         <inertia ixx="0.00005" ixy="0.0" ixz="0.0"
@@ -66,10 +66,10 @@
       <parent link="${prefix}end_effector_link"/>
       <child link="${prefix}gripper_left_upper"/>
-      <origin xyz="0 0 0.04" rpy="0 0 0"/>
+      <origin xyz="0 0.015 0.04" rpy="0 0 0"/>  <!-- Offset to left side -->
     </joint>
     <!-- Left arm - Lower limb (second segment) -->
     <link name="${prefix}gripper_left_lower">
       <visual>
-        <origin xyz="0 0.015 0.03" rpy="0 0 0"/>
+        <origin xyz="0 0 0.03" rpy="0 0 0"/>  <!-- Center of 6cm box -->
         <geometry>
           <box size="0.012 0.018 0.06"/>  <!-- Lower segment, slightly thinner -->
@@ -80,5 +80,5 @@
       </visual>
       <collision>
-        <origin xyz="0 0.015 0.03" rpy="0 0 0"/>
+        <origin xyz="0 0 0.03" rpy="0 0 0"/>
         <geometry>
           <box size="0.012 0.018 0.06"/>
@@ -86,5 +86,5 @@
       </collision>
       <inertial>
-        <origin xyz="0 0.015 0.03" rpy="0 0 0"/>
+        <origin xyz="0 0 0.03" rpy="0 0 0"/>
         <mass value="0.04"/>
         <inertia ixx="0.00004" ixy="0.0" ixz="0.0"
@@ -96,10 +96,10 @@
       <parent link="${prefix}gripper_left_upper"/>
       <child link="${prefix}gripper_left_lower"/>
-      <origin xyz="0 0 0.06" rpy="0 0 0"/>  <!-- Offset from upper limb -->
+      <origin xyz="0 0 0.06" rpy="0 0 0"/>  <!-- At end of upper limb -->
     </joint>
     <!-- Left arm tip (tapered end) -->
     <link name="${prefix}gripper_left_tip">
       <visual>
-        <origin xyz="0 0.015 0.07" rpy="0 0 0"/>
+        <origin xyz="0 0 0.01" rpy="0 0 0"/>  <!-- Center of 2cm box -->
         <geometry>
           <box size="0.01 0.015 0.02"/>  <!-- Smaller tip -->
@@ -110,5 +110,5 @@
       </visual>
       <collision>
-        <origin xyz="0 0.015 0.07" rpy="0 0 0"/>
+        <origin xyz="0 0 0.01" rpy="0 0 0"/>
         <geometry>
           <box size="0.01 0.015 0.02"/>
@@ -124,5 +124,5 @@
     <link name="${prefix}gripper_right_upper">
       <visual>
-        <origin xyz="0 -0.015 0.03" rpy="0 0 0"/>
+        <origin xyz="0 0 0.03" rpy="0 0 0"/>  <!-- Center of this 6cm segment -->
         <geometry>
           <box size="0.015 0.022 0.06"/>  <!-- Upper segment -->
@@ -133,5 +133,5 @@
       </visual>
       <collision>
-        <origin xyz="0 -0.015 0.03" rpy="0 0 0"/>
+        <origin xyz="0 0 0.03" rpy="0 0 0"/>
         <geometry>
           <box size="0.015 0.022 0.06"/>
@@ -139,5 +139,5 @@
       </collision>
       <inertial>
-        <origin xyz="0 -0.015 0.03" rpy="0 0 0"/>
+        <origin xyz="0 0 0.03" rpy="0 0 0"/>
         <mass value="0.05"/>
         <inertia ixx="0.00005" ixy="0.0" ixz="0.0"
@@ -149,10 +149,10 @@
       <parent link="${prefix}end_effector_link"/>
       <child link="${prefix}gripper_right_upper"/>
-      <origin xyz="0 0 0.04" rpy="0 0 0"/>
+      <origin xyz="0 -0.015 0.04" rpy="0 0 0"/>  <!-- Offset to the right -->
     </joint>
     <!-- Right arm - Lower limb (second segment) -->
     <link name="${prefix}gripper_right_lower">
       <visual>
-        <origin xyz="0 -0.015 0.03" rpy="0 0 0"/>
+        <origin xyz="0 0 0.03" rpy="0 0 0"/>  <!-- Center of this 6cm segment -->
         <geometry>
           <box size="0.012 0.018 0.06"/>  <!-- Lower segment, slightly thinner -->
@@ -163,5 +163,5 @@
       </visual>
       <collision>
-        <origin xyz="0 -0.015 0.03" rpy="0 0 0"/>
+        <origin xyz="0 0 0.03" rpy="0 0 0"/>
         <geometry>
           <box size="0.012 0.018 0.06"/>
@@ -169,5 +169,5 @@
       </collision>
       <inertial>
-        <origin xyz="0 -0.015 0.03" rpy="0 0 0"/>
+        <origin xyz="0 0 0.03" rpy="0 0 0"/>
         <mass value="0.04"/>
         <inertia ixx="0.00004" ixy="0.0" ixz="0.0"
@@ -179,10 +179,10 @@
       <parent link="${prefix}gripper_right_upper"/>
       <child link="${prefix}gripper_right_lower"/>
-      <origin xyz="0 0 0.06" rpy="0 0 0"/>  <!-- Offset from upper limb -->
+      <origin xyz="0 0 0.06" rpy="0 0 0"/>  <!-- At end of upper limb -->
     </joint>
     <!-- Right arm tip (tapered end) -->
     <link name="${prefix}gripper_right_tip">
       <visual>
-        <origin xyz="0 -0.015 0.07" rpy="0 0 0"/>
+        <origin xyz="0 0 0.01" rpy="0 0 0"/>  <!-- Center of 2cm tip -->
         <geometry>
           <box size="0.01 0.015 0.02"/>  <!-- Smaller tip -->
@@ -193,5 +193,5 @@
       </visual>
       <collision>
-        <origin xyz="0 -0.015 0.07" rpy="0 0 0"/>
+        <origin xyz="0 0 0.01" rpy="0 0 0"/>
         <geometry>
           <box size="0.01 0.015 0.02"/>
