Commit message: working gripper

File: ros2_system/src/motion_control_module/urdf/end_effector.urdf.xacro (robot description, xacro)
@@ -3,34 +3,34 @@
   <!--
     End-effector attachment for UR5e
-    Tongs/Scissors-style gripper with two prongs
+    Uses actual gripper mesh model
   -->
   <xacro:macro name="end_effector" params="prefix">
-    <!-- Base/Pivot link (connection point) -->
+    <!-- Gripper link with STL mesh -->
     <link name="${prefix}end_effector_link">
+      <!-- Gripper mesh scaled from mm to meters -->
       <visual>
-        <origin xyz="0 0 0.02" rpy="0 0 0"/>
+        <origin xyz="0 0 0" rpy="3.14159 0 0"/>  <!-- Flipped 180 degrees around X axis -->
         <geometry>
-          <!-- Base mount - small cylinder -->
-          <cylinder radius="0.025" length="0.04"/>
+          <mesh filename="package://motion_control_module/meshes/gripper.stl" scale="0.001 0.001 0.001"/>
         </geometry>
-        <material name="base_material">
-          <color rgba="0.2 0.2 0.2 1.0"/>  <!-- Dark gray -->
+        <material name="gripper_material">
+          <color rgba="0.7 0.7 0.7 1.0"/>  <!-- Light gray -->
         </material>
       </visual>
       <collision>
-        <origin xyz="0 0 0.02" rpy="0 0 0"/>
+        <origin xyz="0 0 0" rpy="3.14159 0 0"/>  <!-- Flipped 180 degrees around X axis -->
         <geometry>
-          <cylinder radius="0.025" length="0.04"/>
+          <mesh filename="package://motion_control_module/meshes/gripper.stl" scale="0.001 0.001 0.001"/>
         </geometry>
       </collision>
       <inertial>
         <origin xyz="0 0 0.05" rpy="0 0 0"/>
-        <mass value="0.3"/>
-        <inertia ixx="0.0005" ixy="0.0" ixz="0.0"
-                 iyy="0.0005" iyz="0.0"
-                 izz="0.0005"/>
+        <mass value="0.5"/>
+        <inertia ixx="0.001" ixy="0.0" ixz="0.0"
+                 iyy="0.001" iyz="0.0"
+                 izz="0.001"/>
       </inertial>
     </link>
-    <!-- Joint connecting tool0 to end-effector base -->
+    <!-- Joint connecting tool0 to end-effector -->
     <joint name="${prefix}end_effector_joint" type="fixed">
       <parent link="${prefix}tool0"/>
@@ -38,176 +38,10 @@
       <origin xyz="0 0 0" rpy="0 0 0"/>
     </joint>
-    <!-- Left arm - Upper limb (first segment) -->
-    <link name="${prefix}gripper_left_upper">
-      <visual>
-        <origin xyz="0 0 0.03" rpy="0 0 0"/>  <!-- Center of 6cm box -->
-        <geometry>
-          <box size="0.015 0.022 0.06"/>  <!-- Upper segment -->
-        </geometry>
-        <material name="prong_material">
-          <color rgba="0.7 0.7 0.7 1.0"/>  <!-- Light gray -->
-        </material>
-      </visual>
-      <collision>
-        <origin xyz="0 0 0.03" rpy="0 0 0"/>
-        <geometry>
-          <box size="0.015 0.022 0.06"/>
-        </geometry>
-      </collision>
-      <inertial>
-        <origin xyz="0 0 0.03" rpy="0 0 0"/>
-        <mass value="0.05"/>
-        <inertia ixx="0.00005" ixy="0.0" ixz="0.0"
-                 iyy="0.00005" iyz="0.0"
-                 izz="0.000005"/>
-      </inertial>
-    </link>
-    <joint name="${prefix}gripper_left_upper_joint" type="fixed">
-      <parent link="${prefix}end_effector_link"/>
-      <child link="${prefix}gripper_left_upper"/>
-      <origin xyz="0 0.015 0.04" rpy="0 0 0"/>  <!-- Offset to left side -->
-    </joint>
-    <!-- Left arm - Lower limb (second segment) -->
-    <link name="${prefix}gripper_left_lower">
-      <visual>
-        <origin xyz="0 0 0.03" rpy="0 0 0"/>  <!-- Center of 6cm box -->
-        <geometry>
-          <box size="0.012 0.018 0.06"/>  <!-- Lower segment, slightly thinner -->
-        </geometry>
-        <material name="prong_material">
-          <color rgba="0.7 0.7 0.7 1.0"/>  <!-- Light gray -->
-        </material>
-      </visual>
-      <collision>
-        <origin xyz="0 0 0.03" rpy="0 0 0"/>
-        <geometry>
-          <box size="0.012 0.018 0.06"/>
-        </geometry>
-      </collision>
-      <inertial>
-        <origin xyz="0 0 0.03" rpy="0 0 0"/>
-        <mass value="0.04"/>
-        <inertia ixx="0.00004" ixy="0.0" ixz="0.0"
-                 iyy="0.00004" iyz="0.0"
-                 izz="0.000004"/>
-      </inertial>
-    </link>
-    <joint name="${prefix}gripper_left_lower_joint" type="fixed">
-      <parent link="${prefix}gripper_left_upper"/>
-      <child link="${prefix}gripper_left_lower"/>
-      <origin xyz="0 0 0.06" rpy="0 0 0"/>  <!-- At end of upper limb -->
-    </joint>
-    <!-- Left arm tip (tapered end) -->
-    <link name="${prefix}gripper_left_tip">
-      <visual>
-        <origin xyz="0 0 0.01" rpy="0 0 0"/>  <!-- Center of 2cm box -->
-        <geometry>
-          <box size="0.01 0.015 0.02"/>  <!-- Smaller tip -->
-        </geometry>
-        <material name="tip_material">
-          <color rgba="0.5 0.5 0.5 1.0"/>  <!-- Medium gray -->
-        </material>
-      </visual>
-      <collision>
-        <origin xyz="0 0 0.01" rpy="0 0 0"/>
-        <geometry>
-          <box size="0.01 0.015 0.02"/>
-        </geometry>
-      </collision>
-    </link>
-    <joint name="${prefix}gripper_left_tip_joint" type="fixed">
-      <parent link="${prefix}gripper_left_lower"/>
-      <child link="${prefix}gripper_left_tip"/>
-      <origin xyz="0 0 0.06" rpy="0 0 0"/>  <!-- At end of lower limb -->
-    </joint>
-    <!-- Right arm - Upper limb (first segment) -->
-    <link name="${prefix}gripper_right_upper">
-      <visual>
-        <origin xyz="0 0 0.03" rpy="0 0 0"/>  <!-- Center of this 6cm segment -->
-        <geometry>
-          <box size="0.015 0.022 0.06"/>  <!-- Upper segment -->
-        </geometry>
-        <material name="prong_material">
-          <color rgba="0.7 0.7 0.7 1.0"/>  <!-- Light gray -->
-        </material>
-      </visual>
-      <collision>
-        <origin xyz="0 0 0.03" rpy="0 0 0"/>
-        <geometry>
-          <box size="0.015 0.022 0.06"/>
-        </geometry>
-      </collision>
-      <inertial>
-        <origin xyz="0 0 0.03" rpy="0 0 0"/>
-        <mass value="0.05"/>
-        <inertia ixx="0.00005" ixy="0.0" ixz="0.0"
-                 iyy="0.00005" iyz="0.0"
-                 izz="0.000005"/>
-      </inertial>
-    </link>
-    <joint name="${prefix}gripper_right_upper_joint" type="fixed">
-      <parent link="${prefix}end_effector_link"/>
-      <child link="${prefix}gripper_right_upper"/>
-      <origin xyz="0 -0.015 0.04" rpy="0 0 0"/>  <!-- Offset to the right -->
-    </joint>
-    <!-- Right arm - Lower limb (second segment) -->
-    <link name="${prefix}gripper_right_lower">
-      <visual>
-        <origin xyz="0 0 0.03" rpy="0 0 0"/>  <!-- Center of this 6cm segment -->
-        <geometry>
-          <box size="0.012 0.018 0.06"/>  <!-- Lower segment, slightly thinner -->
-        </geometry>
-        <material name="prong_material">
-          <color rgba="0.7 0.7 0.7 1.0"/>  <!-- Light gray -->
-        </material>
-      </visual>
-      <collision>
-        <origin xyz="0 0 0.03" rpy="0 0 0"/>
-        <geometry>
-          <box size="0.012 0.018 0.06"/>
-        </geometry>
-      </collision>
-      <inertial>
-        <origin xyz="0 0 0.03" rpy="0 0 0"/>
-        <mass value="0.04"/>
-        <inertia ixx="0.00004" ixy="0.0" ixz="0.0"
-                 iyy="0.00004" iyz="0.0"
-                 izz="0.000004"/>
-      </inertial>
-    </link>
-    <joint name="${prefix}gripper_right_lower_joint" type="fixed">
-      <parent link="${prefix}gripper_right_upper"/>
-      <child link="${prefix}gripper_right_lower"/>
-      <origin xyz="0 0 0.06" rpy="0 0 0"/>  <!-- At end of upper limb -->
-    </joint>
-    <!-- Right arm tip (tapered end) -->
-    <link name="${prefix}gripper_right_tip">
-      <visual>
-        <origin xyz="0 0 0.01" rpy="0 0 0"/>  <!-- Center of 2cm tip -->
-        <geometry>
-          <box size="0.01 0.015 0.02"/>  <!-- Smaller tip -->
-        </geometry>
-        <material name="tip_material">
-          <color rgba="0.5 0.5 0.5 1.0"/>  <!-- Medium gray -->
-        </material>
-      </visual>
-      <collision>
-        <origin xyz="0 0 0.01" rpy="0 0 0"/>
-        <geometry>
-          <box size="0.01 0.015 0.02"/>
-        </geometry>
-      </collision>
-    </link>
-    <joint name="${prefix}gripper_right_tip_joint" type="fixed">
-      <parent link="${prefix}gripper_right_lower"/>
-      <child link="${prefix}gripper_right_tip"/>
-      <origin xyz="0 0 0.06" rpy="0 0 0"/>  <!-- At end of lower limb -->
-    </joint>
-    <!-- Tip frame for easy reference (center between prongs) -->
+    <!-- Tip frame for easy reference (adjust position based on actual gripper dimensions) -->
     <link name="${prefix}end_effector_tip"/>
     <joint name="${prefix}end_effector_tip_joint" type="fixed">
       <parent link="${prefix}end_effector_link"/>
       <child link="${prefix}end_effector_tip"/>
-      <origin xyz="0 0 0.18" rpy="0 0 0"/>  <!-- 18cm from tool0 -->
+      <origin xyz="0 0 0.15" rpy="0 0 0"/>  <!-- Adjust Z value based on gripper length -->
     </joint>
   </xacro:macro>

Commit message: Set up for Tuesday

File: ros2_system/src/motion_control_module/urdf/end_effector.urdf.xacro (robot description, xacro)
@@ -10,5 +10,5 @@
       <!-- Gripper mesh scaled from mm to meters -->
       <visual>
-        <origin xyz="0 0 0" rpy="3.14159 0 0"/>  <!-- Flipped 180 degrees around X axis -->
+        <origin xyz="0 0 0" rpy="3.14159 0 1.5708"/>  <!-- Flipped 180 degrees around X axis, 90 degrees around Z axis -->
         <geometry>
           <mesh filename="package://motion_control_module/meshes/gripper.stl" scale="0.001 0.001 0.001"/>
@@ -19,5 +19,5 @@
       </visual>
       <collision>
-        <origin xyz="0 0 0" rpy="3.14159 0 0"/>  <!-- Flipped 180 degrees around X axis -->
+        <origin xyz="0 0 0" rpy="3.14159 0 1.5708"/>  <!-- Flipped 180 degrees around X axis, 90 degrees around Z axis -->
         <geometry>
           <mesh filename="package://motion_control_module/meshes/gripper.stl" scale="0.001 0.001 0.001"/>
