Commit message: try 1

File: ros2_system/src/motion_control_package/urdf/end_effector.urdf.xacro (robot description, xacro)
@@ -12,5 +12,5 @@
         <origin xyz="0 0 0" rpy="3.14159 0 1.5708"/>  <!-- Flipped 180 degrees around X axis, 90 degrees around Z axis -->
         <geometry>
-          <mesh filename="package://motion_control_module/meshes/gripper.stl" scale="0.001 0.001 0.001"/>
+          <mesh filename="package://motion_control_package/meshes/gripper.stl" scale="0.001 0.001 0.001"/>
         </geometry>
         <material name="gripper_material">
@@ -21,5 +21,5 @@
         <origin xyz="0 0 0" rpy="3.14159 0 1.5708"/>  <!-- Flipped 180 degrees around X axis, 90 degrees around Z axis -->
         <geometry>
-          <mesh filename="package://motion_control_module/meshes/gripper.stl" scale="0.001 0.001 0.001"/>
+          <mesh filename="package://motion_control_package/meshes/gripper.stl" scale="0.001 0.001 0.001"/>
         </geometry>
       </collision>

File: ros2_system/src/motion_control_package/urdf/ur5e_with_end_effector.urdf.xacro (robot description, xacro)
@@ -85,5 +85,5 @@
    </xacro:ur_robot>
    <!-- Include end effector -->
-   <xacro:include filename="$(find motion_control_module)/urdf/gripper.urdf"/>
+   <xacro:include filename="$(find motion_control_package)/urdf/gripper.urdf"/>
    <!-- Coupler between arm and end effector -->
    <joint name="ur5e_gripper_coupler_joint" type="fixed">
